File: multiple_tile-panel.brd (EAGLE design)
At the start: 91.4 x 84.5 mm, 18 parts

Commit message: repanelize - v3
Other:
- board size 91.4 x 84.5 mm -> 91.4 x 81.9 mm
Changed lines of the file:
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@@
 <plain>
 <hole x="38.1" y="38.5572" drill="3.175"/>
-<hole x="58.42" y="38.5572" drill="3.175"/>
-<hole x="38.1" y="75.7428" drill="3.175"/>
 <hole x="58.42" y="75.7428" drill="3.175"/>
 <hole x="38.735" y="64.77" drill="6"/>
@@
 <hole x="48.26" y="50.8" drill="6"/>
 <hole x="57.785" y="50.8" drill="6"/>
-<wire x1="33.02" y1="-0.635" x2="33.02" y2="83.82" width="0.254" layer="20"/>
-<wire x1="33.02" y1="35.56" x2="124.46" y2="35.56" width="0.254" layer="102"/>
+<wire x1="33.02" y1="1.905" x2="33.02" y2="83.82" width="0.254" layer="20"/>
 <wire x1="38.735" y1="64.77" x2="57.785" y2="64.77" width="0.6096" layer="51"/>
 <wire x1="39.37" y1="50.8" x2="48.26" y2="50.8" width="0.6096" layer="51" style="shortdash"/>
@@
 <rectangle x1="44.2722" y1="45.1358" x2="51.8922" y2="45.166275" layer="51"/>
 <hole x="68.58" y="38.5572" drill="3.175"/>
-<hole x="88.9" y="38.5572" drill="3.175"/>
-<hole x="68.58" y="75.7428" drill="3.175"/>
 <hole x="88.9" y="75.7428" drill="3.175"/>
 <wire x1="33.02" y1="83.82" x2="124.46" y2="83.82" width="0.254" layer="20"/>
@@
 <hole x="78.74" y="50.8" drill="6"/>
 <hole x="88.265" y="50.8" drill="6"/>
-<wire x1="124.46" y1="-0.635" x2="33.02" y2="-0.635" width="0.254" layer="20"/>
+<wire x1="124.46" y1="1.905" x2="33.02" y2="1.905" width="0.254" layer="20"/>
 <wire x1="69.215" y1="64.77" x2="88.265" y2="64.77" width="0.6096" layer="51"/>
 <wire x1="69.85" y1="50.8" x2="78.74" y2="50.8" width="0.6096" layer="51" style="shortdash"/>
@@
 <rectangle x1="74.7522" y1="45.1358" x2="82.3722" y2="45.166275" layer="51"/>
 <hole x="99.06" y="38.5572" drill="3.175"/>
-<hole x="119.38" y="38.5572" drill="3.175"/>
-<hole x="99.06" y="75.7428" drill="3.175"/>
 <hole x="119.38" y="75.7428" drill="3.175"/>
 <hole x="99.695" y="64.77" drill="6"/>
@@
 <hole x="109.22" y="50.8" drill="6"/>
 <hole x="118.745" y="50.8" drill="6"/>
-<wire x1="124.46" y1="83.82" x2="124.46" y2="-0.635" width="0.254" layer="20"/>
+<wire x1="124.46" y1="83.82" x2="124.46" y2="1.905" width="0.254" layer="20"/>
 <wire x1="99.695" y1="64.77" x2="118.745" y2="64.77" width="0.6096" layer="51"/>
 <wire x1="100.33" y1="50.8" x2="109.22" y2="50.8" width="0.6096" layer="51" style="shortdash"/>
@@
 <rectangle x1="105.2322" y1="45.10531875" x2="112.8522" y2="45.1358" layer="51"/>
 <rectangle x1="105.2322" y1="45.1358" x2="112.8522" y2="45.166275" layer="51"/>
-<wire x1="63.5" y1="83.82" x2="63.5" y2="-0.635" width="0.254" layer="102"/>
-<wire x1="93.98" y1="83.82" x2="93.98" y2="-0.635" width="0.254" layer="102"/>
-<wire x1="33.02" y1="6.35" x2="124.46" y2="6.35" width="0.254" layer="102"/>
-<wire x1="33.02" y1="78.74" x2="124.46" y2="78.74" width="0.254" layer="102"/>
+<wire x1="33.02" y1="35.56" x2="124.46" y2="35.56" width="0.4064" layer="102"/>
+<wire x1="33.02" y1="78.74" x2="124.46" y2="78.74" width="0.4064" layer="102"/>
+<wire x1="33.02" y1="6.985" x2="124.46" y2="6.985" width="0.4064" layer="102"/>
+<wire x1="63.5" y1="1.905" x2="63.5" y2="83.82" width="0.4064" layer="102"/>
+<wire x1="93.98" y1="1.905" x2="93.98" y2="83.82" width="0.4064" layer="102"/>
 </plain>
 <attributes>
